File: binarybox-barrel.sch (EAGLE design)
At the start: 29 parts, among them IC2 MAX7219CNG, X1 USBPTH

Commit message: cleaned up usb board and arduino sketch
Connections:
- net CLK: now also U$10.3; no longer U$10.4
- net INP10: now also U$10.20/A6; no longer U$10.18/A4
- net INP20: now also U$10.21/A7; no longer U$10.19/A5
- net INP40: now also U$10.22/A8; no longer U$10.20/A6
- net INP80: now also U$10.23/A9; no longer U$10.21/A7
- net LOAD: now also U$10.4; no longer U$10.3
- net MODE01: now also U$10.19/A5; no longer U$10.23/A9
- net MODE02: now also U$10.18/A4; no longer U$10.22/A8
Changed lines of the file:
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@@
 <instance part="LED-MODE02" gate="G$1" x="-12.7" y="0"/>
 <instance part="U$13" gate="G$1" x="-10.16" y="33.02"/>
-<instance part="X1" gate="G$1" x="5.08" y="-43.18" rot="R90"/>
+<instance part="X1" gate="G$1" x="5.08" y="-40.64" rot="R90"/>
 </instances>
 <busses>
@@
 </segment>
 <segment>
+<wire x1="2.54" y1="-43.18" x2="2.54" y2="-55.88" width="0.1524" layer="91"/>
 <pinref part="X1" gate="G$1" pin="VBUS"/>
-<wire x1="2.54" y1="-45.72" x2="2.54" y2="-53.34" width="0.1524" layer="91"/>
 </segment>
 <segment>
@@
 </segment>
 <segment>
+<wire x1="5.08" y1="-43.18" x2="5.08" y2="-55.88" width="0.1524" layer="91"/>
+<wire x1="5.08" y1="-55.88" x2="7.62" y2="-55.88" width="0.1524" layer="91"/>
 <pinref part="X1" gate="G$1" pin="GND"/>
-<wire x1="5.08" y1="-45.72" x2="5.08" y2="-53.34" width="0.1524" layer="91"/>
 </segment>
 <segment>
@@
 </segment>
 <segment>
-<pinref part="U$10" gate="G$1" pin="4"/>
-<wire x1="76.2" y1="-63.5" x2="81.28" y2="-63.5" width="0.1524" layer="91"/>
+<pinref part="U$10" gate="G$1" pin="3"/>
+<wire x1="76.2" y1="-66.04" x2="81.28" y2="-66.04" width="0.1524" layer="91"/>
+<label x="81.28" y="-66.04" size="1.778" layer="95" xref="yes"/>
 </segment>
 </net>
@@
 </segment>
 <segment>
-<pinref part="U$10" gate="G$1" pin="3"/>
-<wire x1="76.2" y1="-66.04" x2="81.28" y2="-66.04" width="0.1524" layer="91"/>
+<pinref part="U$10" gate="G$1" pin="4"/>
+<wire x1="76.2" y1="-63.5" x2="81.28" y2="-63.5" width="0.1524" layer="91"/>
+<label x="81.28" y="-63.5" size="1.778" layer="95" xref="yes"/>
 </segment>
 </net>
@@
 <pinref part="U$10" gate="G$1" pin="2"/>
 <wire x1="76.2" y1="-68.58" x2="81.28" y2="-68.58" width="0.1524" layer="91"/>
+<label x="81.28" y="-68.58" size="1.778" layer="95" xref="yes"/>
 </segment>
 </net>
@@
 </segment>
 <segment>
-<pinref part="U$10" gate="G$1" pin="23/A9"/>
-<wire x1="45.72" y1="-63.5" x2="38.1" y2="-63.5" width="0.1524" layer="91"/>
-<label x="38.1" y="-63.5" size="1.778" layer="95" rot="R180" xref="yes"/>
+<pinref part="U$10" gate="G$1" pin="19/A5"/>
+<wire x1="45.72" y1="-53.34" x2="30.48" y2="-53.34" width="0.1524" layer="91"/>
+<label x="30.48" y="-53.34" size="1.778" layer="95" rot="R180" xref="yes"/>
 </segment>
 </net>
@@
 </segment>
 <segment>
-<pinref part="U$10" gate="G$1" pin="22/A8"/>
-<wire x1="45.72" y1="-60.96" x2="38.1" y2="-60.96" width="0.1524" layer="91"/>
-<label x="38.1" y="-60.96" size="1.778" layer="95" rot="R180" xref="yes"/>
+<pinref part="U$10" gate="G$1" pin="18/A4"/>
+<wire x1="45.72" y1="-50.8" x2="30.48" y2="-50.8" width="0.1524" layer="91"/>
+<label x="30.48" y="-50.8" size="1.778" layer="95" rot="R180" xref="yes"/>
 </segment>
 </net>
@@
 </segment>
 <segment>
-<pinref part="U$10" gate="G$1" pin="18/A4"/>
-<wire x1="45.72" y1="-50.8" x2="30.48" y2="-50.8" width="0.1524" layer="91"/>
-<label x="30.48" y="-50.8" size="1.778" layer="95" rot="R180" xref="yes"/>
+<pinref part="U$10" gate="G$1" pin="20/A6"/>
+<wire x1="45.72" y1="-55.88" x2="30.48" y2="-55.88" width="0.1524" layer="91"/>
+<label x="30.48" y="-55.88" size="1.778" layer="95" rot="R180" xref="yes"/>
 </segment>
 </net>
@@
 </segment>
 <segment>
-<pinref part="U$10" gate="G$1" pin="19/A5"/>
-<wire x1="45.72" y1="-53.34" x2="30.48" y2="-53.34" width="0.1524" layer="91"/>
-<label x="30.48" y="-53.34" size="1.778" layer="95" rot="R180" xref="yes"/>
+<pinref part="U$10" gate="G$1" pin="21/A7"/>
+<wire x1="45.72" y1="-58.42" x2="30.48" y2="-58.42" width="0.1524" layer="91"/>
+<label x="30.48" y="-58.42" size="1.778" layer="95" rot="R180" xref="yes"/>
 </segment>
 </net>
@@
 </segment>
 <segment>
-<pinref part="U$10" gate="G$1" pin="20/A6"/>
-<wire x1="45.72" y1="-55.88" x2="30.48" y2="-55.88" width="0.1524" layer="91"/>
-<label x="30.48" y="-55.88" size="1.778" layer="95" rot="R180" xref="yes"/>
+<pinref part="U$10" gate="G$1" pin="22/A8"/>
+<wire x1="45.72" y1="-60.96" x2="38.1" y2="-60.96" width="0.1524" layer="91"/>
+<label x="38.1" y="-60.96" size="1.778" layer="95" rot="R180" xref="yes"/>
 </segment>
 </net>
@@
 </segment>
 <segment>
-<pinref part="U$10" gate="G$1" pin="21/A7"/>
-<wire x1="45.72" y1="-58.42" x2="30.48" y2="-58.42" width="0.1524" layer="91"/>
-<label x="30.48" y="-58.42" size="1.778" layer="95" rot="R180" xref="yes"/>
+<pinref part="U$10" gate="G$1" pin="23/A9"/>
+<wire x1="45.72" y1="-63.5" x2="38.1" y2="-63.5" width="0.1524" layer="91"/>
+<label x="38.1" y="-63.5" size="1.778" layer="95" rot="R180" xref="yes"/>
 </segment>
 </net>
@@
 </segment>
 </net>
-<net name="N$8" class="0">
-<segment>
-<wire x1="-30.48" y1="-38.1" x2="-17.78" y2="-38.1" width="0.1524" layer="91"/>
-</segment>
-</net>
